Commit message: modified gripper positions and orientations

File: youbot_common/youbot_description/urdf/youbot_gripper/gripper.urdf.xacro (robot description, xacro)
@@ -51,5 +51,5 @@
 			</inertial>
 			<visual>
-				<origin xyz="0 0 0" rpy="0 0 0" />
+				<origin xyz="0 -0.01 0" rpy="0 0 ${M_PI}" />
 				<geometry>
 					<mesh filename="package://youbot_description/meshes/youbot_gripper/finger.stl" />
@@ -58,5 +58,5 @@
 			</visual>
 			<collision>
-				<origin xyz="0 0 0" rpy="0 0 0" />
+				<origin xyz="0 -0.01 0" rpy="0 0 ${M_PI}" />
 				<geometry>
 					<!--<box size="0.014 0.020 0.046"/>-->
@@ -81,5 +81,5 @@
 			</inertial>
 			<visual>
-				<origin xyz="0 0 0" rpy="0 0 0" />
+				<origin xyz="0 -0.01 0" rpy="0 0 ${M_PI}" />
 				<geometry>
 					<mesh filename="package://youbot_description/meshes/youbot_gripper/finger.stl" />
@@ -88,5 +88,5 @@
 			</visual>
 			<collision>
-				<origin xyz="0.000 0 0" rpy="0 0 0" />
+				<origin xyz="0.000 -0.01 0" rpy="0 0 ${M_PI}" />
 				<geometry>
 					<!--<box size="0.014 0.020 0.046"/>-->

Commit message: rotate gripper to original orientation

File: youbot_common/youbot_description/urdf/youbot_gripper/gripper.urdf.xacro (robot description, xacro)
@@ -51,5 +51,5 @@
 			</inertial>
 			<visual>
-				<origin xyz="0 -0.01 0" rpy="0 0 ${M_PI}" />
+				<origin xyz="0 0 0" rpy="0 0 0" />
 				<geometry>
 					<mesh filename="package://youbot_description/meshes/youbot_gripper/finger.stl" />
@@ -58,5 +58,5 @@
 			</visual>
 			<collision>
-				<origin xyz="0 -0.01 0" rpy="0 0 ${M_PI}" />
+				<origin xyz="0 0 0" rpy="0 0 0" />
 				<geometry>
 					<!--<box size="0.014 0.020 0.046"/>-->
@@ -81,5 +81,5 @@
 			</inertial>
 			<visual>
-				<origin xyz="0 -0.01 0" rpy="0 0 ${M_PI}" />
+				<origin xyz="0 0 0" rpy="0 0 0" />
 				<geometry>
 					<mesh filename="package://youbot_description/meshes/youbot_gripper/finger.stl" />
@@ -88,5 +88,5 @@
 			</visual>
 			<collision>
-				<origin xyz="0.000 -0.01 0" rpy="0 0 ${M_PI}" />
+				<origin xyz="0.000 0 0" rpy="0 0 0" />
 				<geometry>
 					<!--<box size="0.014 0.020 0.046"/>-->

Commit message: modified gripper opening

File: youbot_common/youbot_description/urdf/youbot_gripper/gripper.urdf.xacro (robot description, xacro)
@@ -51,5 +51,5 @@
 			</inertial>
 			<visual>
-				<origin xyz="0 0 0" rpy="0 0 0" />
+				<origin xyz="0 -0.01 0" rpy="0 0 0" />
 				<geometry>
 					<mesh filename="package://youbot_description/meshes/youbot_gripper/finger.stl" />
@@ -58,5 +58,5 @@
 			</visual>
 			<collision>
-				<origin xyz="0 0 0" rpy="0 0 0" />
+				<origin xyz="0 -0.01 0" rpy="0 0 0" />
 				<geometry>
 					<!--<box size="0.014 0.020 0.046"/>-->
@@ -81,5 +81,5 @@
 			</inertial>
 			<visual>
-				<origin xyz="0 0 0" rpy="0 0 0" />
+				<origin xyz="0 -0.01 0" rpy="0 0 0" />
 				<geometry>
 					<mesh filename="package://youbot_description/meshes/youbot_gripper/finger.stl" />
@@ -88,5 +88,5 @@
 			</visual>
 			<collision>
-				<origin xyz="0.000 0 0" rpy="0 0 0" />
+				<origin xyz="0.000 -0.01 0" rpy="0 0 0" />
 				<geometry>
 					<!--<box size="0.014 0.020 0.046"/>-->
