Commit message: include kinect and webcam into urdf

File: youbot_common/youbot_description/robots/youbot.urdf.xacro (robot description, xacro)
@@ -14,4 +14,8 @@
   <!-- youbot arm -->
   <include filename="$(find youbot_description)/urdf/youbot_arm/arm.urdf.xacro"/>
+  <!-- camera -->
+  <include filename="$(find youbot_description)/urdf/sensors/camera.urdf.xacro"/>
+  <!-- kinect -->
+  <include filename="$(find youbot_description)/urdf/sensors/kinect.urdf.xacro"/>
   <!-- youbot gripper -->
   <include filename="$(find youbot_description)/urdf/youbot_gripper/gripper.urdf.xacro" />
@@ -39,3 +43,11 @@
     <origin xyz="0 0 0" rpy="0 0 0" />
   </xacro:youbot_gripper>
+  <!-- camera mounted on arm -->
+  <xacro:youbot_camera name="camera" parent="arm_link_5" ros_topic="camera">
+    <origin xyz="0.075 0 0" rpy="0 -0.65 0" />
+  </xacro:youbot_camera>
+  <!-- kinect mounted on plate -->
+  <xacro:youbot_kinect name="openni" parent="plate_link" ros_topic="kinect">
+    <origin xyz="0 0 0.52" rpy="0 0 0" />
+  </xacro:youbot_kinect>
 </robot>

Commit message: Changed camera position to fron of base

File: youbot_common/youbot_description/robots/youbot.urdf.xacro (robot description, xacro)
@@ -44,6 +44,6 @@
   </xacro:youbot_gripper>
   <!-- camera mounted on arm -->
-  <xacro:youbot_camera name="camera" parent="arm_link_5" ros_topic="camera">
-    <origin xyz="0.075 0 0" rpy="0 -0.65 0" />
+  <xacro:youbot_camera name="camera" parent="base_link" ros_topic="camera">
+    <origin xyz="0.26 0.0 0.05" rpy="0 0 0" />
   </xacro:youbot_camera>
   <!-- kinect mounted on plate -->

Commit message: translated and rotated kinect

File: youbot_common/youbot_description/robots/youbot.urdf.xacro (robot description, xacro)
@@ -49,5 +49,5 @@
   <!-- kinect mounted on plate -->
   <xacro:youbot_kinect name="openni" parent="plate_link" ros_topic="kinect">
-    <origin xyz="0 0 0.52" rpy="0 0 0" />
+    <origin xyz="-0.06 0 0.52" rpy="0 1.57 0" />
   </xacro:youbot_kinect>
 </robot>

Commit message: fixed kinect urdf

File: youbot_common/youbot_description/robots/youbot.urdf.xacro (robot description, xacro)
@@ -49,5 +49,5 @@
   <!-- kinect mounted on plate -->
   <xacro:youbot_kinect name="openni" parent="plate_link" ros_topic="kinect">
-    <origin xyz="-0.06 0 0.52" rpy="0 1.57 0" />
+    <origin xyz="-0.06 0 0.52" rpy="0 0 0" />
   </xacro:youbot_kinect>
 </robot>

File: youbot_common/youbot_description/urdf/sensors/kinect.urdf.xacro (robot description, xacro)
@@ -7,8 +7,12 @@
   <include filename="$(find youbot_description)/urdf/sensors/kinect.gazebo.xacro" />
   <xacro:macro name="youbot_kinect" params="name parent *origin ros_topic">
-    <joint name="${name}_joint" type="fixed">
+    <joint name="${name}_joint" type="revolute">
       <insert_block name="origin" />
       <parent link="${parent}"/>
       <child link="${name}_link"/>
+      <axis xyz="0 -1 0"/>
+      <calibration rising="0"/>
+      <dynamics damping="25.0" friction="10.0"/>
+      <limit effort="100" lower="-0.54" upper="0.54" velocity="1.0"/>
     </joint>
     <link name="${name}_link">
@@ -19,5 +23,5 @@
       </inertial>
       <visual>
-        <origin xyz="0 0 0.015" rpy="0 0 0" />
+        <origin xyz="0 0 0.015" rpy="0 1.5708 0" />
         <geometry>
           <box size="0.02 0.02 0.075"/>
@@ -26,5 +30,5 @@
       </visual>
       <collision>
-        <origin xyz="0 0 0.015" rpy="0 0 0" />
+        <origin xyz="0 0 0.015" rpy="0 1.5708 0" />
         <geometry>
            <box size="0.02 0.02 0.075"/>
@@ -33,5 +37,5 @@
     </link>
     <joint name="${name}_camera_joint" type="fixed">
-      <origin xyz="0 0 0" rpy="1.5708 -1.5708 0" />
+      <origin xyz="0 0 0" rpy="0 0 0" />
       <parent link="${name}_link"/>
       <child link="${name}_camera"/>

Commit message: kinect has no movable joint anymore and publishes on other topic

File: youbot_common/youbot_description/robots/youbot.urdf.xacro (robot description, xacro)
@@ -48,6 +48,6 @@
   </xacro:youbot_camera>
   <!-- kinect mounted on plate -->
-  <xacro:youbot_kinect name="openni" parent="plate_link" ros_topic="kinect">
-    <origin xyz="-0.06 0 0.52" rpy="0 0 0" />
+  <xacro:youbot_kinect name="openni" parent="plate_link" ros_topic="/camera/depth/points1">
+    <origin xyz="-0.06 0 0.6" rpy="0 0.45 0" />
   </xacro:youbot_kinect>
 </robot>

File: youbot_common/youbot_description/urdf/sensors/kinect.urdf.xacro (robot description, xacro)
@@ -7,12 +7,8 @@
   <include filename="$(find youbot_description)/urdf/sensors/kinect.gazebo.xacro" />
   <xacro:macro name="youbot_kinect" params="name parent *origin ros_topic">
-    <joint name="${name}_joint" type="revolute">
+    <joint name="${name}_joint" type="fixed">
       <insert_block name="origin" />
       <parent link="${parent}"/>
       <child link="${name}_link"/>
-      <axis xyz="0 -1 0"/>
-      <calibration rising="0"/>
-      <dynamics damping="25.0" friction="10.0"/>
-      <limit effort="100" lower="-0.54" upper="0.54" velocity="1.0"/>
     </joint>
     <link name="${name}_link">
